File: KiCad/jRobot-Leonardo-Nano/Arduino-UNO.kicad_sch (KiCad schematic)
At the start: 1 part

Commit message: leonardo
Parts:
- removed A?: Arduino_UNO_R3, Module:Arduino_UNO_R3, symbol MCU_Module:Arduino_UNO_R3
- added A3: Arduino_Nano_v3.x, My_Arduino:Arduino_Nano_WithMountingHoles_larger, symbol MCU_Module:Arduino_Nano_v3.x
Connections:
- net +3V3: now also A3.17 (3V3)
- net +5V: now also A3.27 (+5V)
- net A0: now also A3.19 (A0)
- net A1: now also A3.20 (A1)
- net A2: now also A3.21 (A2)
- net A3: now also A3.22 (A3)
- net AREF: now also A3.18 (AREF)
- net D0/Rx: now also A3.2 (D0/RX)
- net D10: now also A3.13 (D10)
- net D11: now also A3.14 (D11)
- net D12: now also A3.15 (D12)
- net D13: now also A3.16 (D13)
- net D1/Tx: now also A3.1 (D1/TX)
- net D2: now also A3.5 (D2)
- net D3: now also A3.6 (D3)
- net D4: now also A3.7 (D4)
- net D5: now also A3.8 (D5)
- net D6: now also A3.9 (D6)
- net D7: now also A3.10 (D7)
- net D8: now also A3.11 (D8)
- net D9: now also A3.12 (D9)
- net GND: now also A3.29 (GND), A3.4 (GND)
- net SCL/A5: now also A3.24 (A5)
- net SDA/A4: now also A3.23 (A4)
- net VCC: now also A3.30 (VIN)
- net ~{RESET}: now also A3.3 (~{RESET})
- new net A6: A3.25 (A6)
- new net A7: A3.26 (A7)
