File: KiCad/jRobot-Micro/jRobot-Micro.kicad_sch (KiCad schematic)
At the start: 27 parts, among them J1 2-pin_power_input_header, M1 Arm, M2 Motor_Servo, M3 Left, M4 Right, U1 ESP-01, U2 AMS1117-5.0, U3 MPU-6050, U4 BSS138, U5 AMS1117-3.3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

Commit message: arduino micro
Connections:
- net D2 renamed D6/A7
- net D3 renamed D9/A9
- net SCL/A5 renamed D3/SCL
- net SDA/A4 renamed D2/SDA
Other:
- removed sheet Arduino UNO
- added sheet ArduinoMicro (ArduinoMicro.kicad_sch)
- moved on the sheet: U3, U6
